File: PCB/Hellboard.kicad_sch (KiCad schematic)
At the start: 32 parts, among them J1 OLED-128x64, Q1 AO3400A, U1 rp2040-zero

Commit message: add datasheets
Parts:
- D2: Datasheet Socket (none) -> http://www.kailh.com/product/Ms/rcb/CPG151101S11-16.pdf
Changed lines of the file:
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@@
 			)
 		)
-		(property "Datasheet" ""
+		(property "Datasheet" "https://www.waveshare.com/rp2040-zero.htm"
 			(at 102.87 44.45 0)
 			(effects
@@
 			)
 		)
-		(property "Description" ""
+		(property "Description" "Waveshare RP2040-Zero controller"
 			(at 93.98 49.53 0)
 			(effects
@@
 			)
 		)
-		(property "Datasheet" ""
+		(property "Datasheet" "https://www.datasheethub.com/ssd1306-128x64-mono-0-96-inch-i2c-oled-display/"
 			(at 160.02 73.66 90)
 			(effects
@@
 			)
 		)
-		(property "Datasheet" "M93C66-WMN6P"
+		(property "Datasheet" "https://www.st.com/resource/en/datasheet/m93c46-w.pdf"
 			(at 232.41 34.29 0)
 			(effects
@@
 			(at 102.87 147.32 0)
 			(effects
+				(font
+					(size 1.27 1.27)
+				)
+				(hide yes)
+			)
+		)
+		(property "Datasheet Socket" "http://www.kailh.com/product/Ms/rcb/CPG151101S11-16.pdf"
+			(at 102.87 147.32 0)
+			(effects
